Commit message: Almost have it all loaded in!

File: sr_common-melodic-devel/sr_description/mujoco_models/urdfs/ur10.urdf (robot description, URDF)
Before this commit: robot ursr, 11 links, 10 joints
Links:
- link ra_base_link: geometry collision mesh filename=/home/osboxes/universal_robot/ur_description/meshes/ur10/co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; visual mesh filename=/home/osboxes/universal_robot/ur_description/meshes/ur10/vi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
- link ra_forearm_link: geometry collision mesh filename=/home/osboxes/universal_robot/ur_description/meshes/ur10/co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; visual mesh filename=/home/osboxes/universal_robot/ur_description/meshes/ur10/vi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
- link ra_shoulder_link: geometry collision mesh filename=/home/osboxes/universal_robot/ur_description/meshes/ur10/co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; visual mesh filename=/home/osboxes/universal_robot/ur_description/meshes/ur10/vi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
- link ra_upper_arm_link: geometry collision mesh filename=/home/osboxes/universal_robot/ur_description/meshes/ur10/co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; visual mesh filename=/home/osboxes/universal_robot/ur_description/meshes/ur10/vi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
- link ra_wrist_1_link: geometry collision mesh filename=/home/osboxes/universal_robot/ur_description/meshes/ur10/co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; visual mesh filename=/home/osboxes/universal_robot/ur_description/meshes/ur10/vi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
- link ra_wrist_2_link: geometry collision mesh filename=/home/osboxes/universal_robot/ur_description/meshes/ur10/co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; visual mesh filename=/home/osboxes/universal_robot/ur_description/meshes/ur10/vi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
- link ra_wrist_3_link: geometry collision mesh filename=/home/osboxes/universal_robot/ur_description/meshes/ur10/co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; visual mesh filename=/home/osboxes/universal_robot/ur_description/meshes/ur10/vi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

File: sr_common-melodic-devel/sr_description/mujoco_models/urdfs/ur10_hand.urdf (robot description, URDF)
Before this commit: robot ur10srh, 43 links, 42 joints
Links:
- link ra_base_link: geometry collision mesh filename=/home/osboxes/universal_robot/ur_description/meshes/ur10/co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; visual mesh filename=/home/osboxes/universal_robot/ur_description/meshes/ur10/vi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
- link ra_forearm_link: geometry collision mesh filename=/home/osboxes/universal_robot/ur_description/meshes/ur10/co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; visual mesh filename=/home/osboxes/universal_robot/ur_description/meshes/ur10/vi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
- link ra_shoulder_link: geometry collision mesh filename=/home/osboxes/universal_robot/ur_description/meshes/ur10/co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; visual mesh filename=/home/osboxes/universal_robot/ur_description/meshes/ur10/vi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
- link ra_upper_arm_link: geometry collision mesh filename=/home/osboxes/universal_robot/ur_description/meshes/ur10/co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; visual mesh filename=/home/osboxes/universal_robot/ur_description/meshes/ur10/vi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
- link ra_wrist_1_link: geometry collision mesh filename=/home/osboxes/universal_robot/ur_description/meshes/ur10/co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; visual mesh filename=/home/osboxes/universal_robot/ur_description/meshes/ur10/vi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
- link ra_wrist_2_link: geometry collision mesh filename=/home/osboxes/universal_robot/ur_description/meshes/ur10/co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; visual mesh filename=/home/osboxes/universal_robot/ur_description/meshes/ur10/vi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
- link ra_wrist_3_link: geometry collision mesh filename=/home/osboxes/universal_robot/ur_description/meshes/ur10/co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; visual mesh filename=/home/osboxes/universal_robot/ur_description/meshes/ur10/vi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
- link rh_ffdistal: geometry collision mesh filename=/home/osboxes/piano-man/sr_common-melodic-devel/sr_descript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 scale=0.001 0.001 0.001; visual mesh filename=/home/osboxes/piano-man/sr_common-melodic-devel/sr_descript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 scale=0.001 0.001 0.001
- link rh_ffknuckle: geometry collision cylinder length=0.014 radius=0.007; visual mesh filename=/home/osboxes/piano-man/sr_common-melodic-devel/sr_descript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 scale=0.001 0.001 0.001
- link rh_ffmiddle: geometry collision cylinder length=0.025 radius=0.007; visual mesh filename=/home/osboxes/piano-man/sr_common-melodic-devel/sr_descript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 scale=0.001 0.001 0.001
- link rh_ffproximal: geometry collision cylinder length=0.040 radius=0.007; visual mesh filename=/home/osboxes/piano-man/sr_common-melodic-devel/sr_descript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 scale=0.001 0.001 0.001
- link rh_forearm: geometry collision mesh filename=/home/osboxes/piano-man/sr_common-melodic-devel/sr_descript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 scale=1 1 1; visual mesh filename=/home/osboxes/piano-man/sr_common-melodic-devel/sr_descript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 scale=0.001 0.001 0.001
- link rh_lfdistal: geometry collision mesh filename=/home/osboxes/piano-man/sr_common-melodic-devel/sr_descript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 scale=0.001 0.001 0.001; visual mesh filename=/home/osboxes/piano-man/sr_common-melodic-devel/sr_descript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 scale=0.001 0.001 0.001
- link rh_lfknuckle: geometry collision cylinder length=0.014 radius=0.007; visual mesh filename=/home/osboxes/piano-man/sr_common-melodic-devel/sr_descript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 scale=0.001 0.001 0.001
- link rh_lfmetacarpal: geometry collision box size=0.018 0.024 0.040; visual mesh filename=/home/osboxes/piano-man/sr_common-melodic-devel/sr_descript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 scale=0.001 0.001 0.001
- link rh_lfmiddle: geometry collision cylinder length=0.025 radius=0.007; visual mesh filename=/home/osboxes/piano-man/sr_common-melodic-devel/sr_descript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 scale=0.001 0.001 0.001
- link rh_lfproximal: geometry collision cylinder length=0.040 radius=0.007; visual mesh filename=/home/osboxes/piano-man/sr_common-melodic-devel/sr_descript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 scale=0.001 0.001 0.001
- link rh_mfdistal: geometry collision mesh filename=/home/osboxes/piano-man/sr_common-melodic-devel/sr_descript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 scale=0.001 0.001 0.001; visual mesh filename=/home/osboxes/piano-man/sr_common-melodic-devel/sr_descript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 scale=0.001 0.001 0.001
- link rh_mfknuckle: geometry collision cylinder length=0.014 radius=0.007; visual mesh filename=/home/osboxes/piano-man/sr_common-melodic-devel/sr_descript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 scale=0.001 0.001 0.001
- link rh_mfmiddle: geometry collision cylinder length=0.025 radius=0.007; visual mesh filename=/home/osboxes/piano-man/sr_common-melodic-devel/sr_descript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 scale=0.001 0.001 0.001
- link rh_mfproximal: geometry collision cylinder length=0.040 radius=0.007; visual mesh filename=/home/osboxes/piano-man/sr_common-melodic-devel/sr_descript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 scale=0.001 0.001 0.001
- link rh_palm: geometry collision box size=0.062 0.007 0.098; visual mesh filename=/home/osboxes/piano-man/sr_common-melodic-devel/sr_descript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 scale=0.001 0.001 0.001
- link rh_rfdistal: geometry collision mesh filename=/home/osboxes/piano-man/sr_common-melodic-devel/sr_descript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 scale=0.001 0.001 0.001; visual mesh filename=/home/osboxes/piano-man/sr_common-melodic-devel/sr_descript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 scale=0.001 0.001 0.001
- link rh_rfknuckle: geometry collision cylinder length=0.014 radius=0.007; visual mesh filename=/home/osboxes/piano-man/sr_common-melodic-devel/sr_descript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 scale=0.001 0.001 0.001
- link rh_rfmiddle: geometry collision cylinder length=0.025 radius=0.007; visual mesh filename=/home/osboxes/piano-man/sr_common-melodic-devel/sr_descript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 scale=0.001 0.001 0.001
- link rh_rfproximal: geometry collision cylinder length=0.040 radius=0.007; visual mesh filename=/home/osboxes/piano-man/sr_common-melodic-devel/sr_descript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 scale=0.001 0.001 0.001
- link rh_thdistal: geometry collision mesh filename=/home/osboxes/piano-man/sr_common-melodic-devel/sr_descript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 scale=0.001 0.001 0.001; visual mesh filename=/home/osboxes/piano-man/sr_common-melodic-devel/sr_descript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 scale=0.001 0.001 0.001
- link rh_thmiddle: geometry collision cylinder length=0.018 radius=0.011; visual mesh filename=/home/osboxes/piano-man/sr_common-melodic-devel/sr_descript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 scale=0.001 0.001 0.001
- link rh_thproximal: geometry collision cylinder length=0.018 radius=0.012; visual mesh filename=/home/osboxes/piano-man/sr_common-melodic-devel/sr_descript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 scale=0.001 0.001 0.001
- link rh_wrist: geometry collision cylinder length=0.030 radius=0.0135; visual mesh filename=/home/osboxes/piano-man/sr_common-melodic-devel/sr_descript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 scale=0.001 0.001 0.001
